File: hardware/link_teensy_fpga/link_teensy_fpga.kicad_sch (KiCad schematic)
At the start: 41 parts, among them J11 2x3, J3 Conn_01x04_Voltage, P1 J1B1211CCD, U1 Teensy4.1, U3 DM-OLED096-636, U30 TXU0202, U32 TXU0102, U33 SN74LVC1G06, U34 SN74LVC1G06, U35 SN74LVC1G06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

Commit message: start fpga adapter
Parts:
- removed R30, R32: 10k, Resistor_SMD:R_0603_1608Metric_Pad0.98x0.95mm_HandSolder, symbol Device:R_Small
- removed U30: TXU0202, Package_SO:VSSOP-8_2.3x2mm_P0.5mm, symbol Transputer:TXU0202
- removed U32: TXU0102, Package_SO:VSSOP-8_2.3x2mm_P0.5mm, symbol Transputer:TXU0102
Connections:
- net Tennsy30 is gone; now on net RESET: U1.22 (30_CRX3)
- net Tennsy31 is gone; now on net ANALYZE: U1.23 (31_CTX3)
- net Tennsy28: now also D3.2 (A), L11.4 (LinkIn), R9.1
- net Tennsy29: now also R111.1

Commit message: Test rev ${VCSSHORTHASH}
Parts:
- removed C50, C51, C52, C53, C54, C56, C57: 0.1µF, Capacitor_SMD:C_0603_1608Metric_Pad1.08x0.95mm_HandSolder, symbol Device:C
- removed C500: 100µF, Capacitor_SMD:CP_Elec_5x3.9, symbol Device:C_Polarized
- removed D3: 1N4148, Diode_SMD:D_SOD-323_HandSoldering, symbol Diode:1N4148
- removed J11: 2x3, Connector_PinHeader_2.54mm:PinHeader_2x03_P2.54mm_Vertical, symbol Connector_Generic:Conn_02x03_Odd_Even
- removed J3: Conn_01x04_Voltage, Connector_PinHeader_2.54mm:PinHeader_1x04_P2.54mm_Vertical, symbol Transputer:Conn_01x04_Voltage
- removed JP14: Jumper_2_Open, Connector_PinHeader_2.54mm:PinHeader_1x02_P2.54mm_Vertical, symbol Jumper:Jumper_2_Open
- removed L11: ~, Connector_IDC:IDC-Header_2x05_P2.54mm_Horizontal, symbol Transputer:Conn_02x05_Gerlach
- removed R111: 56, Resistor_SMD:R_0603_1608Metric_Pad0.98x0.95mm_HandSolder, symbol Device:R_Small
- removed R35, R9: 10k, Resistor_SMD:R_0603_1608Metric_Pad0.98x0.95mm_HandSolder, symbol Device:R_Small
- removed U33, U34, U35, U40, U41, U42: SN74LVC1G06, Package_TO_SOT_SMD:SOT-23-5_HandSoldering, symbol Transputer:SN74LVC1G06
- added J1: ~, Transputer:PinHeader_2x06_P2.54mm_PMODPeriph2B, symbol Transputer:PMOD_PERIPH_2x6
- added TP1: Cable to 5V on Arty, symbol Connector:TestPoint
- added U4: 74HC04, symbol 74xx:74HC04
- D1: footprint Diode_SMD:D_SMB -> (none)
Connections:
- net +3.3V: now also LED1.A1 (A2), LED1.A2, LED2.A1 (A2), LED2.A2, J1.12 (VCC), J1.6 (VCC), U4.14 (VCC)
- net ANALYZE: now also U4.1, U4.5
- net GND: now also J1.11 (GND), J1.5 (GND), U4.7 (GND)
- net RESET: now also U4.11, U4.3
- net Tennsy28: now also J1.7 (IO5)
- net Tennsy29: now also J1.1 (IO1)
- net at R40.2: now also U4.10
- net at R41.2: now also U4.6
- net at R42.2: now also U4.8
- removed net +5V: D1.1 (K), LED1.A1 (A2), LED1.A2, LED2.A1 (A2), LED2.A2, U1.48 (VIN)
- net +5VL: no longer names the net of D1.2 (A)
- net +5VL: now also TP1.1
- net Tennsy32 renamed Error
- net Error: now also U4.12, U4.9
- new net: D1.1 (K), U1.48 (VIN)
- new net: J1.9 (IO7), U4.13
- new net NotAnalyze: J1.2 (IO2), U4.2
- new net NotReset: J1.8 (IO6), U4.4
- no-connect marks 48 -> 47
Other:
- note added: "https://www.mikrocontroller.net/topic/117594"
- note added: "| Transputer Signal | PMOD pins | PMOD pins | Transputer Signal | | LinkIn | PMOD 1 (JA1) | PMOD 7 (JA7) | LinkOut | | NotAnalyse | PMOD 2 (JA2) | PMOD 8 (JA8) | NotReset | | | PMOD 3 (JA3) | PMOD 9 (JA9) | NotError | | | PMOD 4 (JA4) | PMOD 10 (JA10) | | | | PMOD 5 GND | PMOD 11 GND | | | | PMOD 6 VCC3V3 | PMOD 12 VCC3V3 | |"
- note removed: "Muss der nicht an Noterror"
- moved on the sheet: C1, C30, C300, C31, C32, LED1, LED2, P1, R40, R41, R42, R43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
