File: hardware/link_teensy_fpga/link_teensy_fpga.kicad_sch (KiCad schematic)
At the start: 18 parts, among them P1 J1B1211CCD, U1 Teensy4.1, U3 DM-OLED096-636, U4 74HC04

Commit message: cleanup pluto
Parts:
- removed C31, C32: 0.1µF, Capacitor_SMD:C_0603_1608Metric_Pad1.08x0.95mm_HandSolder, symbol Device:C
- removed LED1, LED2: ~, Transputer:mentor_LED_2, symbol Transputer:Mentor_LED_2
- added C3: 0.1µF, Capacitor_SMD:C_0603_1608Metric_Pad1.08x0.95mm_HandSolder, symbol Device:C
- added D_A1, D_E1, D_P1, D_R1: LED, LED_THT:LED_D3.0mm, symbol Device:LED
- added JP1: Jumper_2_Open, Connector_PinHeader_2.54mm:PinHeader_1x02_P2.54mm_Vertical, symbol Jumper:Jumper_2_Open
- added R5, R6, R7: 10k, Resistor_SMD:R_0603_1608Metric_Pad0.98x0.95mm_HandSolder, symbol Device:R_Small
- C2: renamed from C30; KiLib_Generator (none) -> SMD_2terminal_chip_molded
- C5: renamed from C300; KiLib_Generator (none) -> capacitor/SMD/elec_round_polarized
- D1: value D_Schottky_Small -> PMEG2010ER; footprint (none) -> Diode_SMD:Nexperia_CFP3_SOD-123W
- J1: value ~ -> (none)
- R1: renamed from R40; KiLib_Generator (none) -> SMD_2terminal_chip_molded
- R2: renamed from R41; KiLib_Generator (none) -> SMD_2terminal_chip_molded
- R3: renamed from R43; KiLib_Generator (none) -> SMD_2terminal_chip_molded
- R4: renamed from R42; KiLib_Generator (none) -> SMD_2terminal_chip_molded
- TP1: footprint (none) -> Connector_PinHeader_2.54mm:PinHeader_1x01_P2.54mm_Vertical; KiLib_Generator (none) -> connector/pin_header_socket
- U2: renamed from U4; footprint (none) -> Package_SO:SOIC-14_3.9x8.7mm_P1.27mm; KiLib_Generator (none) -> package/gullwing
Connections:
- net +3.3V: now also C3.1, D_A1.2 (A), D_E1.2 (A), D_P1.2 (A), D_R1.2 (A), JP1.1 (A), R5.2, R6.2, R7.2; no longer J1.12 (VCC), J1.6 (VCC)
- net ANALYZE: now also U2.3, U2.9; no longer U2.1, U2.5
- net Error: now also U2.11; no longer U2.9
- net GND: now also C3.2
- net NotAnalyze: now also U2.4, R5.1; no longer U2.2
- net NotReset: now also U2.2, R6.1; no longer U2.4
- net RESET: now also U2.1, U2.5; no longer U2.11, U2.3
- net at R1.2: now also U2.6; no longer U2.10
- net at R1.1: now also D_R1.1 (K)
- net at R2.1: now also D_A1.1 (K)
- net at R3.1: now also D_P1.1 (K)
- net at R2.2: now also U2.8; no longer U2.6
- net at J1.9 (IO7), U2.13: now also R7.1
- net at R4.1: now also D_E1.1 (K)
- net at R4.2: now also U2.10; no longer U2.8
- new net: J1.12 (VCC), J1.6 (VCC), JP1.2 (B)
Other:
- note removed: "https://www.mikrocontroller.net/topic/117594"
- moved on the sheet: C5, R1, R2, U2C, U2D
