File: hardware/link_teensy_fpga/link_teensy_fpga.kicad_pcb (KiCad board)
At the start: 4 copper layers, 80 x 50 mm, 41 parts, among them J11 2x3, J3 Conn_01x04_Voltage, P1 J1B1211CCD, U1 Teensy4.1, U3 DM-OLED096-636, U30 TXU0202, U32 TXU0102, U33 SN74LVC1G06, U34 SN74LVC1G06, U35 SN74LVC1G06, U40 SN74LVC1G06, U41 SN74LVC1G06, U42 SN74LVC1G06

Commit message: cleanup pluto
Parts:
- removed C30, C31, C32, C50, C51, C52, C53, C54, C56, C57: 0.1µF, Capacitor_SMD:C_0603_1608Metric_Pad1.08x0.95mm_HandSolder
- removed C300, C500: 100µF, Capacitor_SMD:CP_Elec_5x3.9
- removed D3: 1N4148, Diode_SMD:D_SOD-323_HandSoldering
- removed J11: 2x3, Connector_PinHeader_2.54mm:PinHeader_2x03_P2.54mm_Vertical
- removed J3: Conn_01x04_Voltage, Connector_PinHeader_2.54mm:PinHeader_1x04_P2.54mm_Vertical
- removed JP14: Jumper_2_Open, Connector_PinHeader_2.54mm:PinHeader_1x02_P2.54mm_Vertical
- removed L11: ~, Connector_IDC:IDC-Header_2x05_P2.54mm_Horizontal
- removed LED1, LED2: ~, Transputer:mentor_LED_2
- removed R111: 56, Resistor_SMD:R_0603_1608Metric_Pad0.98x0.95mm_HandSolder
- removed R30, R32, R35, R9: 10k, Resistor_SMD:R_0603_1608Metric_Pad0.98x0.95mm_HandSolder
- removed R40, R41, R42, R43: 470, Resistor_SMD:R_0603_1608Metric_Pad0.98x0.95mm_HandSolder
- removed U30: TXU0202, Package_SO:VSSOP-8_2.3x2mm_P0.5mm
- removed U32: TXU0102, Package_SO:VSSOP-8_2.3x2mm_P0.5mm
- removed U33, U34, U35, U40, U41, U42: SN74LVC1G06, Package_TO_SOT_SMD:SOT-23-5_HandSoldering
- added C2: 0.1µF, Capacitor_SMD:C_0603_1608Metric_Pad1.08x0.95mm_HandSolder, F.Cu at (109.8, 107.5)
- added C3: 0.1µF, Capacitor_SMD:C_0603_1608Metric_Pad1.08x0.95mm_HandSolder, F.Cu at (92.2, 125.8)
- added C5: 100µF, Capacitor_SMD:CP_Elec_5x3.9, F.Cu at (115.2, 143.6)
- added D_A1: LED, LED_THT:LED_D3.0mm, F.Cu at (124.7, 134.6)
- added D_E1: LED, LED_THT:LED_D3.0mm, F.Cu at (124.7, 128.6)
- added D_P1: LED, LED_THT:LED_D3.0mm, F.Cu at (124.7, 146.5)
- added D_R1: LED, LED_THT:LED_D3.0mm, F.Cu at (124.7, 140.5)
- added J1: ~, Transputer:PinHeader_2x06_P2.54mm_PMODPeriph2B, F.Cu at (123.3, 109.2)
- added JP1: 3,3V, Connector_PinHeader_2.54mm:PinHeader_1x02_P2.54mm_Vertical, F.Cu at (116.6, 108.2)
- added R1: 470, Resistor_SMD:R_0603_1608Metric_Pad0.98x0.95mm_HandSolder, F.Cu at (121.3, 140.7)
- added R2: 470, Resistor_SMD:R_0603_1608Metric_Pad0.98x0.95mm_HandSolder, F.Cu at (121.3, 134.7)
- added R3: 470, Resistor_SMD:R_0603_1608Metric_Pad0.98x0.95mm_HandSolder, F.Cu at (121.3, 146.6)
- added R4: 470, Resistor_SMD:R_0603_1608Metric_Pad0.98x0.95mm_HandSolder, F.Cu at (121.3, 128.8)
- added R5: 10k, Resistor_SMD:R_0603_1608Metric_Pad0.98x0.95mm_HandSolder, F.Cu at (100.4, 111.7)
- added R6: 10k, Resistor_SMD:R_0603_1608Metric_Pad0.98x0.95mm_HandSolder, F.Cu at (104.7, 111.7)
- added R7: 10k, Resistor_SMD:R_0603_1608Metric_Pad0.98x0.95mm_HandSolder, F.Cu at (115.8, 111.7)
- added TP1: Cable to 5V on Arty, Connector_PinHeader_2.54mm:PinHeader_1x01_P2.54mm_Vertical, F.Cu at (54.9, 127.0)
- added U2: 74HC04, Package_SO:SOIC-14_3.9x8.7mm_P1.27mm, F.Cu at (110.2, 116.8)
- D1: value D_Schottky_Small -> PMEG2010ER; footprint Diode_SMD:D_SMB -> Diode_SMD:Nexperia_CFP3_SOD-123W; moved to F.Cu
- moved U3 25.1 mm to (89.7, 117.8)
- moved C1 11.4 mm to (73.8, 113.4), turned to -90 degrees
- moved D1 8.57 mm to (51.6, 128.3)
- moved P1 2.36 mm to (61.0, 115.6)
- moved U1 2.36 mm to (80.8, 140.2)
Connections:
- net +5V renamed Net-(D1-K)
- D1 pad 2: +5VL -> Net-(D1-A)
- U1 pad 22: /Tennsy30 -> RESET
- U1 pad 23: /Tennsy31 -> ANALYZE
- U1 pad 24: /Tennsy32 -> Error
Routing:
- net +3.3V: track 321.5 -> 26.9 mm, vias 7 -> 3
- net Net-(D1-K): track 242.1 -> 2.87 mm, vias 16 -> 0
- net +5VL: track 93.0 -> 0.00 mm, vias 1 -> 0
- net Error: track 0.00 -> 67.9 mm
- net /Tennsy31: track 48.5 -> 0.00 mm, vias 1 -> 0
- net /Tennsy30: track 36.0 -> 0.00 mm, vias 1 -> 0
- net /NotReset: track 0.00 -> 33.1 mm, vias 0 -> 1
- net ANALYZE: track 22.2 -> 55.2 mm
- net Net-(JP14-B): track 32.7 -> 0.00 mm
- net /NotAnalyze: track 0.00 -> 29.4 mm, vias 0 -> 1
- net Net-(R41-Pad2): track 28.5 -> 0.00 mm, vias 2 -> 0
- net Net-(R1-Pad2): track 0.00 -> 27.7 mm
- net Net-(J11-Pin_3): track 27.5 -> 0.00 mm, vias 1 -> 0
- net Net-(R42-Pad2): track 27.0 -> 0.00 mm, vias 2 -> 0
- net GND: track 36.0 -> 14.6 mm, vias 20 -> 5
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- added copper zone on In2.Cu, net +3.3V
Other:
- board size 80 x 50 mm -> 80 x 45.5 mm
