File: hardware/link_teensy_small/link_teensy_small.kicad_sch (KiCad schematic)
At the start: 41 parts, among them J11 2x3, J3 Conn_01x04_Voltage, P1 J1B1211CCD, U1 Teensy4.1, U3 DM-OLED096-636, U30 TXU0202, U32 TXU0102, U33 SN74LVC1G06, U34 SN74LVC1G06, U35 SN74LVC1G06, U40 SN74LVC1G06, U41 SN74LVC1G06, U42 SN74LVC1G06

Commit message: cleanup pluto
Other:
- title: (none) -> Link Teensy Small
Changed lines of the file:
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@@
 	(paper "A3")
 	(title_block
+		(title "Link Teensy Small")
 		(date "2026-02-21")
+		(rev "01")
 	)
 	(text "Auf Tennsy VIN und VUSB trennen und Schottky-Diode einsetzen"

Commit message: new kicad version
Parts:
- L11, LED1, LED2: value ~ -> (none)
